File: Schematics/Power Amp V1.0/ES.1/MCU.kicad_sch (KiCad schematic)
At the start: 0 parts

Commit message: [Schematics] Power Amp V1.0 ES.1 회로도 업데이트
- M483 MCU 회로 추가
Parts:
- added C1, C4, C5, C7, C8, C9: 0603B104K500, Capacitor_SMD:C_0603_1608Metric, symbol Capacitor_MLCC:0603B104K500
- added C10, C12: 0603X105K6R3, SMC:0603, symbol Capacitor_MLCC:0603X105K6R3
- added C2, C3: 0603N120J500, Capacitor_SMD:C_0603_1608Metric, symbol Capacitor_MLCC:0603N120J500
- added C6: 0603B104K500, SMC:0603, symbol Capacitor_MLCC:0603B104K500
- added J5: Nuvoton_ARM, Debug:TLSR8258_program, symbol Connector_Debug:Nuvoton_ARM
- added R10, R11: WR06X1003FTL, SMR:0603, symbol Resistor:WR06X1003FTL
- added R3: WR06X1002FTL, Resistor_SMD:R_0603_1608Metric, symbol Resistor:WR06X1002FTL
- added R4: WR06W3R30FTL, Resistor_SMD:R_0603_1608Metric, symbol Resistor:WR06W3R30FTL
- added U1: M483SIDAE, LQFP:LQFP64, symbol MCU:M483SIDAE
- added X1: XTL0567-12M000, CRYSTAL:CRSTAL_SMD_3225-4Pin, symbol Crystal:XTL0567-12M000
Connections:
- new net: C12.2, U1.24 (LDO_CAP)
- new net: C10.2, U1.50 (LDO_CAP)
- new net +3.3V: C4.2, C6.2, C7.2, C8.2, C9.2, J5.1 (VDD), R10.2, R11.2, R3.2, R4.2, U1.13 (VDD), U1.23 (VDD), U1.31 (VDDIO), U1.42 (HSUSB_VDD33), U1.51 (VDD)
- new net AVDD: C5.2, R4.1, U1.57 (AVDD)
- new net GND: C1.1, C10.1, C12.1, C2.1, C3.1, C4.1, C5.1, C6.1, C7.1, C8.1, C9.1, J5.5 (GND), U1.22 (VSS), U1.45 (HSUSB_VSS), U1.49 (VSS), U1.59 (AVSS)
- new net NRST: C1.2, J5.4 (RESET), R3.1, U1.32 (nRESET)
- new net OSC_IN: C3.2, U1.16 (PF3), X1.3
- new net OSC_OUT: C2.2, U1.17 (PF2), X1.1
- new net SWCLK: J5.3 (SWCLK), R11.1, U1.34 (PF1/SWCLK)
- new net SWDIO: J5.2 (SWDIO), R10.1, U1.33 (PF0/SWDIO)
