File: Schematics/Power Amp V1.0/ES.1/Speaker Amp.kicad_sch (KiCad schematic)
At the start: 45 parts, among them CN1 WJ2EDGRC-5.08-2P, CN2 WJ2EDGRC-5.08-2P, U3 TAS5756MDCA

Commit message: [Schematics] Power Amp V1.0 ES.1 회로도 업데이트
- M483 MCU 회로 추가
Parts:
- renumbered U3 to U2
Changed lines of the file:
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@@
 		(on_board yes)
 		(dnp no)
-		(property "Reference" "U3"
+		(property "Reference" "U2"
 			(at 133.35 41.91 0)
 			(effects
@@
 			(project "Power Amp"
 				(path "/7c979da8-7e54-461e-8675-99eaf95aeefe/52e364c8-bbc1-4146-9b61-4f56ef4be0ff"
-					(reference "U3")
+					(reference "U2")
 					(unit 1)
 				)
